File: kicad/ReTuLaReMake.kicad_sch (KiCad schematic)
At the start: 26 parts, among them J1 40 Pin DIP Header, J2 Conn_02x05_Odd_Even, J3 Conn_01x01_Male, U1 ATF1508AS-10AU100

Commit message: KiCAD: Add clock filter; adjust decoupling
Parts:
- added C10: 47p, Capacitor_SMD:C_0805_2012Metric_Pad1.18x1.45mm_HandSolder, symbol Device:C_Small
- added R9: 120R, Resistor_SMD:R_0805_2012Metric_Pad1.20x1.40mm_HandSolder, symbol Device:R_Small
- renumbered R9 to R12
Connections:
- net GND: now also C10.1
- net HO2: now also R9.2; no longer U1.85 (I/O/GCLK3)
- new net HO2filtered: C10.2, R9.1, U1.85 (I/O/GCLK3)
Changed lines of the file:
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@@
   (junction (at 91.44 173.99) (diameter 0) (color 0 0 0 0)
+  )
+  (junction (at 232.41 118.11) (diameter 0) (color 0 0 0 0)
   )
   (no_connect (at 114.3 38.1))
@@
     (stroke (width 0) (type default) (color 0 0 0 0))
   )
+  (wire (pts (xy 240.03 118.11) (xy 255.27 118.11))
+    (stroke (width 0) (type default) (color 0 0 0 0))
+  )
+  (wire (pts (xy 232.41 118.11) (xy 232.41 120.65))
+    (stroke (width 0) (type default) (color 0 0 0 0))
+  )
   (wire (pts (xy 215.9 102.87) (xy 215.9 111.76))
     (stroke (width 0) (type default) (color 0 0 0 0))
@@
     (stroke (width 0) (type default) (color 0 0 0 0))
   )
+  (wire (pts (xy 232.41 118.11) (xy 234.95 118.11))
+    (stroke (width 0) (type default) (color 0 0 0 0))
+  )
   (wire (pts (xy 142.24 101.6) (xy 167.64 101.6))
     (stroke (width 0) (type default) (color 0 0 0 0))
@@
     (stroke (width 0) (type default) (color 0 0 0 0))
   )
+  (wire (pts (xy 223.52 118.11) (xy 232.41 118.11))
+    (stroke (width 0) (type default) (color 0 0 0 0))
+  )
   (wire (pts (xy 255.27 102.87) (xy 215.9 102.87))
     (stroke (width 0) (type default) (color 0 0 0 0))
@@
     (effects (font (size 1.27 1.27)) (justify right bottom))
   )
+  (label "HO2filtered" (at 223.52 118.11 180)
+    (effects (font (size 1.27 1.27)) (justify right bottom))
+  )
   (label "VCC" (at 93.98 149.86 270)
     (effects (font (size 1.27 1.27)) (justify right bottom))
@@
     (effects (font (size 1.27 1.27)) (justify left bottom))
   )
-  (label "HO2" (at 111.76 38.1 90)
+  (label "HO2filtered" (at 111.76 38.1 90)
     (effects (font (size 1.27 1.27)) (justify left bottom))
   )
@@
     (pin "2")
   )
+  (symbol (lib_id "power:GND") (at 232.41 125.73 0) (unit 1)
+    (in_bom yes) (on_board yes) (fields_autoplaced)
+    (property "Reference" "#PWR0104" (id 0) (at 232.41 132.08 0)
+      (effects (font (size 1.27 1.27)) hide)
+    )
+    (property "Value" "GND" (id 1) (at 232.41 130.81 0))
+    (property "Footprint" "" (id 2) (at 232.41 125.73 0)
+      (effects (font (size 1.27 1.27)) hide)
+    )
+    (property "Datasheet" "" (id 3) (at 232.41 125.73 0)
+      (effects (font (size 1.27 1.27)) hide)
+    )
+    (pin "1")
+  )
   (symbol (lib_id "Connector_Generic:Conn_02x05_Odd_Even") (at 201.93 146.05 0) (unit 1)
     (in_bom yes) (on_board yes) (fields_autoplaced)
@@
   (symbol (lib_id "Device:R_Small") (at 167.64 104.14 0) (unit 1)
     (in_bom yes) (on_board yes)
-    (property "Reference" "R9" (id 0) (at 170.18 104.14 90))
+    (property "Reference" "R12" (id 0) (at 170.18 104.14 90))
     (property "Value" "NF" (id 1) (at 165.1 104.14 90))
     (property "Footprint" "Resistor_SMD:R_0805_2012Metric_Pad1.20x1.40mm_HandSolder" (id 2) (at 167.64 104.14 0)
@@
     )
     (property "Datasheet" "~" (id 3) (at 203.2 81.28 0)
+      (effects (font (size 1.27 1.27)) hide)
+    )
+    (pin "1")
+    (pin "2")
+  )
+  (symbol (lib_id "Device:C_Small") (at 232.41 123.19 180) (unit 1)
+    (in_bom yes) (on_board yes)
+    (property "Reference" "C10" (id 0) (at 226.06 121.92 0)
+      (effects (font (size 1.27 1.27)) (justify right))
+    )
+    (property "Value" "47p" (id 1) (at 226.06 124.46 0)
+      (effects (font (size 1.27 1.27)) (justify right))
+    )
+    (property "Footprint" "Capacitor_SMD:C_0805_2012Metric_Pad1.18x1.45mm_HandSolder" (id 2) (at 232.41 123.19 0)
+      (effects (font (size 1.27 1.27)) hide)
+    )
+    (property "Datasheet" "~" (id 3) (at 232.41 123.19 0)
       (effects (font (size 1.27 1.27)) hide)
     )
@@
     (pin "2")
   )
+  (symbol (lib_id "Device:R_Small") (at 237.49 118.11 90) (unit 1)
+    (in_bom yes) (on_board yes)
+    (property "Reference" "R9" (id 0) (at 234.95 115.57 90))
+    (property "Value" "120R" (id 1) (at 240.03 115.57 90))
+    (property "Footprint" "Resistor_SMD:R_0805_2012Metric_Pad1.20x1.40mm_HandSolder" (id 2) (at 237.49 118.11 0)
+      (effects (font (size 1.27 1.27)) hide)
+    )
+    (property "Datasheet" "~" (id 3) (at 237.49 118.11 0)
+      (effects (font (size 1.27 1.27)) hide)
+    )
+    (pin "1")
+    (pin "2")
+  )
   (symbol (lib_id "Device:R_Small") (at 203.2 86.36 90) (unit 1)
     (in_bom yes) (on_board yes)
@@
       (reference "#PWR0103") (unit 1) (value "GND") (footprint "")
     )
+    (path "/6f7ecab3-6cf9-49bb-808d-6b8e85fa2a0c"
+      (reference "#PWR0104") (unit 1) (value "GND") (footprint "")
+    )
     (path "/7777a350-903e-40b7-a5ca-d09eb3d07ef4"
       (reference "C1") (unit 1) (value "100n") (footprint "Capacitor_SMD:C_0805_2012Metric_Pad1.18x1.45mm_HandSolder")
@@
       (reference "C9") (unit 1) (value "10u") (footprint "Capacitor_Tantalum_SMD:CP_EIA-6032-28_Kemet-C_Pad2.25x2.35mm_HandSolder")
     )
+    (path "/b33220f7-157a-4f56-ab1a-69cec2ad1943"
+      (reference "C10") (unit 1) (value "47p") (footprint "Capacitor_SMD:C_0805_2012Metric_Pad1.18x1.45mm_HandSolder")
+    )
     (path "/a81c6f94-59da-4c1b-b6ae-b6b190f1e0c4"
       (reference "D1") (unit 1) (value "MBR130") (footprint "Diode_SMD:D_SOD-123")
@@
       (reference "R8") (unit 1) (value "0R") (footprint "Resistor_SMD:R_0805_2012Metric_Pad1.20x1.40mm_HandSolder")
     )
-    (path "/99dba31c-ee68-4162-a785-0f0e83785d19"
-      (reference "R9") (unit 1) (value "NF") (footprint "Resistor_SMD:R_0805_2012Metric_Pad1.20x1.40mm_HandSolder")
+    (path "/d7a48f6d-bb9a-43f5-bb53-5526daab0f91"
+      (reference "R9") (unit 1) (value "120R") (footprint "Resistor_SMD:R_0805_2012Metric_Pad1.20x1.40mm_HandSolder")
     )
     (path "/6df6e71d-43b0-4d40-beec-529e26c51d4b"
@@
       (reference "R11") (unit 1) (value "NF") (footprint "Resistor_SMD:R_0805_2012Metric_Pad1.20x1.40mm_HandSolder")
     )
+    (path "/99dba31c-ee68-4162-a785-0f0e83785d19"
+      (reference "R12") (unit 1) (value "NF") (footprint "Resistor_SMD:R_0805_2012Metric_Pad1.20x1.40mm_HandSolder")
+    )
     (path "/5667c8b7-51f0-4e01-9182-7dd1424c90df"

Commit message: KiCAD: Remove R1-R8
Parts:
- removed R1, R2, R3, R4, R5, R6, R7, R8: 0R, Resistor_SMD:R_0805_2012Metric_Pad1.20x1.40mm_HandSolder, symbol Device:R_Small
- renumbered R9 to R1, R10 to R2, R11 to R3, R12 to R4
Connections:
- net HD0: now also J1.6 (Pin_6)
- net HD1: now also J1.7 (Pin_7)
- net HD2: now also J1.8 (Pin_8)
- net HD3: now also J1.9 (Pin_9)
- net HD4: now also J1.10 (Pin_10)
- net HD5: now also J1.11 (Pin_11)
- net HD6: now also J1.12 (Pin_12)
- net HD7: now also J1.13 (Pin_13)
